File: mainboard.brd (EAGLE design)
At the start: 100 x 80 mm, 10 parts, among them IC1 NE555D, IC2 4051D, IC3 4051D, IC4 4051D, IC5 4051D, IC6 74LS138D, IC7 4053D, IC8 74LS393D, IC9 74LS138D

Commit message: added diodes
Parts:
- added D1, D10, D11, D12, D13, D14, D15, D16, D2, D3, D4, D5, D6, D7, D8, D9: GREEN, SparkFun-LED:LED-0603
- added R1: (no value), SparkFun-Resistors:0603-RES
Connections:
- new net N$11: D1.C, IC6.15
- new net N$12: D2.C, IC6.14
- new net N$13: D3.C, IC6.13
- new net N$14: D4.C, IC6.12
- new net N$15: D5.C, IC6.11
- new net N$16: D6.C, IC6.10
- new net N$17: D7.C, IC6.9
- new net N$18: D8.C, IC6.7
- new net N$19: D9.C, IC9.15
- new net N$20: D10.C, IC9.14
- new net N$21: D11.C, IC9.13
- new net N$22: D12.C, IC9.12
- new net N$23: D13.C, IC9.11
- new net N$24: D14.C, IC9.10
- new net N$25: D15.C, IC9.9
- new net N$26: D16.C, IC9.7
- new net N$27: D1.A, D10.A, D11.A, D12.A, D13.A, D14.A, D15.A, D16.A, D2.A, D3.A, D4.A, D5.A, D6.A, D7.A, D8.A, D9.A, R1.1
- net N$6: now also IC6.4, IC6.5, IC9.6; no longer IC6.6, IC9.4
